File: envsensor/envsensor.kicad_pcb (KiCad board)
At the start: 2 copper layers, 52 x 70 mm, 5 parts, among them U3 SCD30, U4 MS5611-01BA, U5 BH1750

Commit message: added led screen
Parts:
- U1: value ~ -> LD2450
- U4: footprint Library:MS5611 -> Package_LGA:LGA-8_3x5mm_P1.25mm
- U5: footprint Library:Untitled_1 -> Library:BH1750
